File: hw/pcb/4 Battery Swap Shield (4BSS) rev.A/rev.A/4BSS rev.A.sch (EAGLE design)
At the start: 47 parts, among them CN1 1776275-2, CN2 1776275-2, CN3 1776275-2, CN4 1776275-2, CN5 1776275-2, CN6 1776275-2, Q1 MMBT2222A, Q2 MMBT2222A, Q3 MMBT2222A, Q4 MMBT2222A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

Commit message: added BOM and sch in pdf format
Parts:
- C1, C2: VAL (none) -> 100nF
Connections:
- net N$14 renamed BJT_EMITERS
Other:
- note added: "@ Vbat = 13V -> Vadc @ pot max = 13*0.203=2,639V"
- note added: "@ Vbat = 13V -> Vadc @ pot min = 13*0.169=2,197V"
- note added: "Aten center = 110k/(480k+110k)= 0,1864v/v"
- note added: "Hongfa HFD31/5-L2"
- note added: "designed by: J.A.Peral"
- note removed: "@ Vbat = 13V -> Adc con pot a tope 1= 13*0.203=2,639V"
- note removed: "@ Vbat = 13V -> Adc con pot a tope 2= 13*0.169=2,197V"
- moved on the sheet: C1, C2, CN5-1, CN5-2, CN6-1, CN6-2, D5, D6, D7, D8, JP1, JP2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
